Commit message: Sim Step 4: back-projection verified against ground truth; found and fixed depth camera bug (undefined material -> invalid depth on close objects)

File: ros2_ws/src/library_bot_description/urdf/d405_camera.xacro (robot description, xacro)
@@ -33,6 +33,6 @@
   <xacro:property name="d405_height" value="480"/>
   <xacro:property name="d405_update_rate" value="15"/>  <!-- Hz; raise once perf is confirmed -->
-  <xacro:property name="d405_near" value="0.07"/>       <!-- matches datasheet min range -->
-  <xacro:property name="d405_far" value="0.5"/>         <!-- matches datasheet max reliable range -->
+  <xacro:property name="d405_near" value="0.07"/>       <!-- TEMP: widened for debugging, was 0.07 -->
+  <xacro:property name="d405_far" value="0.5"/>          <!-- TEMP: widened for debugging, was 0.5 -->
   <xacro:property name="M_PI" value="3.14159265359"/>
   <xacro:macro name="d405_camera" params="parent xyz:='0 0 0' rpy:='0 0 0'">
@@ -81,4 +81,6 @@
         </camera>
         <plugin name="d405_controller" filename="libgazebo_ros_camera.so">
+          <min_depth>0.05</min_depth>
+          <max_depth>0.6</max_depth>
           <ros>
             <namespace>d405</namespace>

File: ros2_ws/src/library_bot_description/urdf/library_bot.urdf.xacro (robot description, xacro)
@@ -68,3 +68,6 @@
     <origin xyz="0.3 0 0.5" rpy="0 0 0"/>
   </joint>
+  <gazebo reference="test_target_link">
+    <material>Gazebo/Grey</material>
+  </gazebo>
 </robot>

Commit message: Working baseline: Gazebo + MoveIt2 + D405 depth verified

File: ros2_ws/src/library_bot_description/urdf/d405_camera.xacro (robot description, xacro)
@@ -85,9 +85,4 @@
           <ros>
             <namespace>d405</namespace>
-            <remapping>image_raw:=color/image_raw</remapping>
-            <remapping>camera_info:=color/camera_info</remapping>
-            <remapping>depth/image_raw:=depth/image_rect_raw</remapping>
-            <remapping>depth/camera_info:=depth/camera_info</remapping>
-            <remapping>points:=depth/points</remapping>
           </ros>
           <camera_name>d405</camera_name>

File: ros2_ws/src/library_bot_moveit_config/config/library_bot.ros2_control.xacro (robot description, xacro)
@@ -2,17 +2,23 @@
 <robot xmlns:xacro="http://www.ros.org/wiki/xacro">
   <!--
-    ros2_control block using mock_components/GenericSystem.
+    ros2_control block for library_bot.
+    use_sim:=false (default) -> mock_components/GenericSystem: fake hardware
+      that echoes commands back instantly. No Gazebo, no physics. Still
+      used by move_group.launch.py for fast planning-only tests.
+    use_sim:=true            -> gazebo_ros2_control/GazeboSystem: joints are
+      driven inside real Gazebo physics (used by gazebo_moveit.launch.py).
     Real motors (steppers, per the plan doc) aren't wired to ROS2 control
-    yet - this is a placeholder hardware interface so MoveIt2 has something
-    to command and read joint states from in sim, the same "sim placeholder
-    for the eventual real interface" pattern already used for MoveIt2/KDL
-    itself (project plan Section 6.1). Swap this block for a real
-    ros2_control hardware plugin later without touching anything else in
-    this package.
+    yet; swap this block for a real hardware plugin later without touching
+    anything else in this package.
   -->
-  <xacro:macro name="library_bot_ros2_control" params="name:=library_bot">
+  <xacro:macro name="library_bot_ros2_control" params="name:=library_bot use_sim:=false">
     <ros2_control name="${name}" type="system">
       <hardware>
-        <plugin>mock_components/GenericSystem</plugin>
+        <xacro:if value="${use_sim}">
+          <plugin>gazebo_ros2_control/GazeboSystem</plugin>
+        </xacro:if>
+        <xacro:unless value="${use_sim}">
+          <plugin>mock_components/GenericSystem</plugin>
+        </xacro:unless>
       </hardware>
       <joint name="joint1_waist">

File: ros2_ws/src/library_bot_moveit_config/config/library_bot_with_ros2_control.xacro (robot description, xacro)
@@ -4,13 +4,24 @@
   Combines the real robot geometry with the ros2_control hardware
   interface macro (config/library_bot.ros2_control.xacro) so that the
-  robot_description passed to ros2_control_node actually contains a
-  <ros2_control> tag. This lives in library_bot_moveit_config rather than
-  editing library_bot_description's own xacro file directly, keeping the
-  mock-hardware-for-testing concern separate from the robot's real
-  geometry description.
+  robot_description passed to ros2_control actually contains a
+  <ros2_control> tag. Lives in library_bot_moveit_config so the
+  control concern stays separate from the robot's geometry description.
+  Argument:
+    use_sim (default false)
+      false -> mock hardware, no Gazebo plugin (move_group.launch.py)
+      true  -> GazeboSystem + the gazebo_ros2_control plugin that loads
+               ros2_controllers.yaml inside Gazebo (gazebo_moveit.launch.py)
 -->
 <robot name="library_bot" xmlns:xacro="http://www.ros.org/wiki/xacro">
+  <xacro:arg name="use_sim" default="false"/>
   <xacro:include filename="$(find library_bot_description)/urdf/library_bot.urdf.xacro"/>
   <xacro:include filename="$(find library_bot_moveit_config)/config/library_bot.ros2_control.xacro"/>
-  <xacro:library_bot_ros2_control/>
+  <xacro:library_bot_ros2_control use_sim="$(arg use_sim)"/>
+  <xacro:if value="$(arg use_sim)">
+    <gazebo>
+      <plugin filename="libgazebo_ros2_control.so" name="gazebo_ros2_control">
+        <parameters>$(find library_bot_moveit_config)/config/ros2_controllers.yaml</parameters>
+      </plugin>
+    </gazebo>
+  </xacro:if>
 </robot>
