Commit message: Sim Steps 2-3: depth verification, ArUco marker model + live detection working

File: ros2_ws/src/library_bot_description/urdf/library_bot.urdf.xacro (robot description, xacro)
@@ -44,3 +44,27 @@
   </joint>
   <xacro:d405_camera parent="ee_placeholder_link" xyz="0 0 0" rpy="0 0 0"/>
+    <!-- Sim Step 2 test target: a small box placed 0.3m directly in front of
+       the D405 (within its 0.07-0.5m depth range), purely to confirm the
+       depth sensor gives correct, non-garbage distance readings. Not part
+       of the real robot — remove once Step 2 is verified. -->
+  <link name="test_target_link">
+    <visual>
+      <origin xyz="0 0 0" rpy="0 0 0"/>
+      <geometry><box size="0.05 0.1 0.1"/></geometry>
+    </visual>
+    <collision>
+      <origin xyz="0 0 0" rpy="0 0 0"/>
+      <geometry><box size="0.05 0.1 0.1"/></geometry>
+    </collision>
+    <inertial>
+      <mass value="0.01"/>
+      <origin xyz="0 0 0"/>
+      <inertia ixx="1e-6" ixy="0" ixz="0" iyy="1e-6" iyz="0" izz="1e-6"/>
+    </inertial>
+  </link>
+  <joint name="test_target_joint" type="fixed">
+    <parent link="base_link"/>
+    <child link="test_target_link"/>
+    <origin xyz="0.3 0 0.5" rpy="0 0 0"/>
+  </joint>
 </robot>

Commit message: Sim Step 5: hand-eye transform via tf2, remove leftover test_target_link

File: ros2_ws/src/library_bot_description/urdf/library_bot.urdf.xacro (robot description, xacro)
@@ -44,30 +44,3 @@
   </joint>
   <xacro:d405_camera parent="ee_placeholder_link" xyz="0 0 0" rpy="0 0 0"/>
-    <!-- Sim Step 2 test target: a small box placed 0.3m directly in front of
-       the D405 (within its 0.07-0.5m depth range), purely to confirm the
-       depth sensor gives correct, non-garbage distance readings. Not part
-       of the real robot — remove once Step 2 is verified. -->
-  <link name="test_target_link">
-    <visual>
-      <origin xyz="0 0 0" rpy="0 0 0"/>
-      <geometry><box size="0.05 0.1 0.1"/></geometry>
-    </visual>
-    <collision>
-      <origin xyz="0 0 0" rpy="0 0 0"/>
-      <geometry><box size="0.05 0.1 0.1"/></geometry>
-    </collision>
-    <inertial>
-      <mass value="0.01"/>
-      <origin xyz="0 0 0"/>
-      <inertia ixx="1e-6" ixy="0" ixz="0" iyy="1e-6" iyz="0" izz="1e-6"/>
-    </inertial>
-  </link>
-  <joint name="test_target_joint" type="fixed">
-    <parent link="base_link"/>
-    <child link="test_target_link"/>
-    <origin xyz="0.3 0 0.5" rpy="0 0 0"/>
-  </joint>
-  <gazebo reference="test_target_link">
-    <material>Gazebo/Grey</material>
-  </gazebo>
 </robot>

Commit message: Step 6 complete: DH table, sim-appropriate joint limits, MoveIt2/KDL working (3 poses confirmed), consolidated handoff doc; add moveit_config package and world file (previously untracked)

File: ros2_ws/src/library_bot_description/urdf/library_bot.urdf.xacro (robot description, xacro)
@@ -2,19 +2,32 @@
 <robot name="library_bot" xmlns:xacro="http://www.ros.org/wiki/xacro">
   <!--
-    Placeholder robot description. Purpose: give the D405 camera something
-    to mount on so we can verify it actually publishes real topics in
-    Gazebo, before any real arm geometry exists.
-    base_footprint -> base_link -> ee_placeholder_link -> d405_link
-    ee_placeholder_link stands in for wherever the real end-effector /
-    wrist will eventually be, once arm geometry (O1, blocked on the
-    library visit) locks. Nothing downstream depends on its exact
-    position being correct yet.
+    Sim Step 6: real arm kinematic chain.
+    Chain: base_footprint -> base_link -> link1(waist) -> link2(shoulder)
+    -> link3(elbow) -> link4/5/6(spherical wrist) -> ee_link -> D405.
+    RESOLVED (library visit, confirmed):
+      - base_link height off ground = 0.40m (arm mounted on cart)
+      - Big shelf target layers: 0.14m, 0.44m, 0.74m, 1.04m (4 of 6 layers,
+        team decision) - all within reach envelope from shoulder height
+        (0.57m = 0.40 cart + 0.17 motor stack), verified against L1+L2=1.06m.
+      - Shelf depth 61cm, grasp offset 14cm (from earlier torque/offset work).
+    STILL PLACEHOLDER (refine when finalized):
+      - d1 = 0.17m: Nema34+worm gearbox stack estimate, not final CAD.
+      - d4 = 0: assumes wrist sits at end of L2 link; confirm vs forearm design.
+      - Joint limits below are simulation-appropriate estimates, chosen to
+        avoid obvious self-collision given current link geometry (only
+        joint3_elbow was tightened, from +-2.35 to +-2.094 rad) - NOT
+        measured mechanical hardstops. Revisit once the arm is printed and
+        real hardstop angles can be physically tested.
+      - Link visuals/collisions are primitive stand-ins (cylinders), not
+        real link geometry.
+    L1 = L2 = 0.53m: confirmed real arm geometry (Sim Step 5 log).
   -->
   <xacro:include filename="$(find library_bot_description)/urdf/d405_camera.xacro"/>
-  <!-- base_footprint is a standard ROS convention: a massless frame at
-       ground level, directly below base_link, used as the reference
-       point nav2 and other tools expect. base_link itself can then sit
-       up off the ground at the robot's actual body height. -->
   <link name="base_footprint"/>
+  <link name="world"/>
+  <joint name="world_to_base_footprint" type="fixed">
+    <parent link="world"/>
+    <child link="base_footprint"/>
+  </joint>
   <link name="base_link">
     <inertial>
@@ -35,12 +48,118 @@
     <parent link="base_footprint"/>
     <child link="base_link"/>
-    <origin xyz="0 0 0.1" rpy="0 0 0"/>
+    <origin xyz="0 0 0.40" rpy="0 0 0"/>
   </joint>
-  <link name="ee_placeholder_link"/>
-  <joint name="ee_placeholder_joint" type="fixed">
+  <link name="link1">
+    <inertial>
+      <mass value="1.5"/>
+      <origin xyz="0 0 0"/>
+      <inertia ixx="0.01" ixy="0" ixz="0" iyy="0.01" iyz="0" izz="0.01"/>
+    </inertial>
+    <visual>
+      <geometry><cylinder radius="0.06" length="0.1"/></geometry>
+    </visual>
+    <collision>
+      <geometry><cylinder radius="0.06" length="0.1"/></geometry>
+    </collision>
+  </link>
+  <joint name="joint1_waist" type="revolute">
     <parent link="base_link"/>
-    <child link="ee_placeholder_link"/>
-    <origin xyz="0 0 0.5" rpy="0 0 0"/>
+    <child link="link1"/>
+    <origin xyz="0 0 0.17" rpy="0 0 0"/>
+    <axis xyz="0 0 1"/>
+    <limit lower="-3.14" upper="3.14" effort="60" velocity="1.0"/>
   </joint>
-  <xacro:d405_camera parent="ee_placeholder_link" xyz="0 0 0" rpy="0 0 0"/>
+  <link name="link2">
+    <inertial>
+      <mass value="2.0"/>
+      <origin xyz="0.265 0 0"/>
+      <inertia ixx="0.02" ixy="0" ixz="0" iyy="0.02" iyz="0" izz="0.005"/>
+    </inertial>
+    <visual>
+      <origin xyz="0.265 0 0" rpy="0 1.5708 0"/>
+      <geometry><cylinder radius="0.04" length="0.53"/></geometry>
+    </visual>
+    <collision>
+      <origin xyz="0.265 0 0" rpy="0 1.5708 0"/>
+      <geometry><cylinder radius="0.04" length="0.53"/></geometry>
+    </collision>
+  </link>
+  <joint name="joint2_shoulder" type="revolute">
+    <parent link="link1"/>
+    <child link="link2"/>
+    <origin xyz="0 0 0" rpy="-1.5708 0 0"/>
+    <axis xyz="0 0 1"/>
+    <limit lower="-1.57" upper="1.57" effort="80" velocity="1.0"/>
+  </joint>
+  <link name="link3">
+    <inertial>
+      <mass value="1.5"/>
+      <origin xyz="0.265 0 0"/>
+      <inertia ixx="0.015" ixy="0" ixz="0" iyy="0.015" iyz="0" izz="0.004"/>
+    </inertial>
+    <visual>
+      <origin xyz="0.265 0 0" rpy="0 1.5708 0"/>
+      <geometry><cylinder radius="0.035" length="0.53"/></geometry>
+    </visual>
+    <collision>
+      <origin xyz="0.265 0 0" rpy="0 1.5708 0"/>
+      <geometry><cylinder radius="0.035" length="0.53"/></geometry>
+    </collision>
+  </link>
+  <joint name="joint3_elbow" type="revolute">
+    <parent link="link2"/>
+    <child link="link3"/>
+    <origin xyz="0.53 0 0" rpy="0 0 0"/>
+    <axis xyz="0 0 1"/>
+    <limit lower="-2.094" upper="2.094" effort="40" velocity="1.0"/>
+  </joint>
+  <link name="link4">
+    <inertial>
+      <mass value="0.4"/>
+      <origin xyz="0 0 0"/>
+      <inertia ixx="0.002" ixy="0" ixz="0" iyy="0.002" iyz="0" izz="0.002"/>
+    </inertial>
+    <visual><geometry><cylinder radius="0.03" length="0.06"/></geometry></visual>
+    <collision><geometry><cylinder radius="0.03" length="0.06"/></geometry></collision>
+  </link>
+  <joint name="joint4_wrist1" type="revolute">
+    <parent link="link3"/>
+    <child link="link4"/>
+    <origin xyz="0.53 0 0" rpy="-1.5708 0 0"/>
+    <axis xyz="0 0 1"/>
+    <limit lower="-3.14" upper="3.14" effort="15" velocity="1.5"/>
+  </joint>
+  <link name="link5">
+    <inertial>
+      <mass value="0.3"/>
+      <origin xyz="0 0 0"/>
+      <inertia ixx="0.0015" ixy="0" ixz="0" iyy="0.0015" iyz="0" izz="0.0015"/>
+    </inertial>
+    <visual><geometry><cylinder radius="0.025" length="0.05"/></geometry></visual>
+    <collision><geometry><cylinder radius="0.025" length="0.05"/></geometry></collision>
+  </link>
+  <joint name="joint5_wrist2" type="revolute">
+    <parent link="link4"/>
+    <child link="link5"/>
+    <origin xyz="0 0 0" rpy="1.5708 0 0"/>
+    <axis xyz="0 0 1"/>
+    <limit lower="-2.09" upper="2.09" effort="15" velocity="1.5"/>
+  </joint>
+  <link name="ee_link">
+    <inertial>
+      <mass value="0.2"/>
+      <origin xyz="0 0 0"/>
+      <inertia ixx="0.001" ixy="0" ixz="0" iyy="0.001" iyz="0" izz="0.001"/>
+    </inertial>
+    <visual><geometry><cylinder radius="0.02" length="0.04"/></geometry></visual>
+    <collision><geometry><cylinder radius="0.02" length="0.04"/></geometry></collision>
+  </link>
+  <joint name="joint6_wrist3" type="revolute">
+    <parent link="link5"/>
+    <child link="ee_link"/>
+    <origin xyz="0 0 0" rpy="-1.5708 0 0"/>
+    <axis xyz="0 0 1"/>
+    <limit lower="-3.14" upper="3.14" effort="15" velocity="1.5"/>
+  </joint>
+  <xacro:d405_camera parent="ee_link" xyz="0.05 0 0" rpy="0 0 0"/>
 </robot>

Commit message: Camera-guided pick and place between two tables by marker ID: scripts, models, gripper, vendored attach plugin (with local patch), MoveIt config, tools

File: ros2_ws/src/library_bot_description/urdf/library_bot.urdf.xacro (robot description, xacro)
@@ -162,4 +162,6 @@
     <limit lower="-3.14" upper="3.14" effort="15" velocity="1.5"/>
   </joint>
-  <xacro:d405_camera parent="ee_link" xyz="0.05 0 0" rpy="0 0 0"/>
+  <xacro:include filename="$(find library_bot_description)/urdf/gripper.xacro"/>
+  <xacro:parallel_gripper parent="ee_link"/>
+  <xacro:d405_camera parent="ee_link" xyz="0.03 0 -0.045" rpy="0 0 0"/>
 </robot>

File: ros2_ws/src/library_bot_moveit_config/config/library_bot.ros2_control.xacro (robot description, xacro)
@@ -29,10 +29,14 @@
       <joint name="joint2_shoulder">
         <command_interface name="position"/>
-        <state_interface name="position"/>
+        <state_interface name="position">
+          <param name="initial_value">-0.8495</param>
+        </state_interface>
         <state_interface name="velocity"/>
       </joint>
       <joint name="joint3_elbow">
         <command_interface name="position"/>
-        <state_interface name="position"/>
+        <state_interface name="position">
+          <param name="initial_value">1.699</param>
+        </state_interface>
         <state_interface name="velocity"/>
       </joint>
@@ -44,5 +48,7 @@
       <joint name="joint5_wrist2">
         <command_interface name="position"/>
-        <state_interface name="position"/>
+        <state_interface name="position">
+          <param name="initial_value">-0.8495</param>
+        </state_interface>
         <state_interface name="velocity"/>
       </joint>
@@ -52,4 +58,30 @@
         <state_interface name="velocity"/>
       </joint>
+      <joint name="finger_left_joint">
+        <xacro:if value="${use_sim}">
+          <command_interface name="effort">
+            <param name="min">-40</param>
+            <param name="max">40</param>
+          </command_interface>
+        </xacro:if>
+        <xacro:unless value="${use_sim}">
+          <command_interface name="position"/>
+        </xacro:unless>
+        <state_interface name="position"/>
+        <state_interface name="velocity"/>
+      </joint>
+      <joint name="finger_right_joint">
+        <xacro:if value="${use_sim}">
+          <command_interface name="effort">
+            <param name="min">-40</param>
+            <param name="max">40</param>
+          </command_interface>
+        </xacro:if>
+        <xacro:unless value="${use_sim}">
+          <command_interface name="position"/>
+        </xacro:unless>
+        <state_interface name="position"/>
+        <state_interface name="velocity"/>
+      </joint>
     </ros2_control>
   </xacro:macro>
